File: hw/usb-rgb.sch (KiCad schematic (older format))
At the start: 12 parts, among them J1 Conn_01x05_Female, J2 USB_B_Micro, U1 SAMD11D14A-M, U2 MCP1700-3302E_SOT23

Commit message: 🏁 pcb race entry
Parts:
- C1, C2: footprint (none) -> Capacitor_SMD:C_0603_1608Metric_Pad1.05x0.95mm_HandSolder
- J1: footprint (none) -> kicadlib:SMD_JST_5_PIN_VERT
- J2: footprint (none) -> kicadlib:usb_micro_b_smt
- R1, R2, R3: footprint (none) -> Resistor_SMD:R_0603_1608Metric_Pad1.05x0.95mm_HandSolder
- TP1, TP2: footprint (none) -> kicadlib:TEST_0.100
Changed lines of the file:
@@
 $EndDescr
-$Comp
-L Regulator_Linear:MCP1700-3302E_SOT23 U2
-U 1 1 5BA6934A
-P 5400 1550
-F 0 "U2" H 5400 1792 50  0000 C CNN
-F 1 "MCP1700-3302E_SOT23" H 5400 1701 50  0000 C CNN
-F 2 "Package_TO_SOT_SMD:SOT-23" H 5400 1775 50  0001 C CNN
-F 3 "http://ww1.microchip.com/downloads/en/DeviceDoc/20001826C.pdf" H 5400 1550 50  0001 C CNN
-	1    5400 1550
-	1    0    0    -1
-$EndComp
 $Comp
 L MCU_Microchip_SAMD:SAMD11D14A-M U1
@@
 F 0 "J2" H 2705 2567 50  0000 C CNN
 F 1 "USB_B_Micro" H 2705 2476 50  0000 C CNN
-F 2 "" H 2800 2050 50  0001 C CNN
+F 2 "kicadlib:usb_micro_b_smt" H 2800 2050 50  0001 C CNN
 F 3 "~" H 2800 2050 50  0001 C CNN
 	1    2650 2100
@@
 F 0 "C2" H 5915 1846 50  0000 L CNN
 F 1 "C" H 5915 1755 50  0000 L CNN
-F 2 "" H 5838 1650 50  0001 C CNN
+F 2 "Capacitor_SMD:C_0603_1608Metric_Pad1.05x0.95mm_HandSolder" H 5838 1650 50  0001 C CNN
 F 3 "~" H 5800 1800 50  0001 C CNN
 	1    5800 1800
@@
 F 0 "TP2" H 6708 3470 50  0000 L CNN
 F 1 "TestPoint" H 6708 3379 50  0000 L CNN
-F 2 "" H 6850 3350 50  0001 C CNN
+F 2 "kicadlib:TEST_0.100" H 6850 3350 50  0001 C CNN
 F 3 "~" H 6850 3350 50  0001 C CNN
 	1    6650 3350
@@
 F 0 "R1" V 6393 4750 50  0000 C CNN
 F 1 "R" V 6484 4750 50  0000 C CNN
-F 2 "" V 6530 4750 50  0001 C CNN
+F 2 "Resistor_SMD:R_0603_1608Metric_Pad1.05x0.95mm_HandSolder" V 6530 4750 50  0001 C CNN
 F 3 "~" H 6600 4750 50  0001 C CNN
 	1    6600 4750
@@
 F 0 "R2" V 6400 4850 50  0000 C CNN
 F 1 "R22" V 6500 4850 50  0000 C CNN
-F 2 "" V 6530 4850 50  0001 C CNN
+F 2 "Resistor_SMD:R_0603_1608Metric_Pad1.05x0.95mm_HandSolder" V 6530 4850 50  0001 C CNN
 F 3 "~" H 6600 4850 50  0001 C CNN
 	1    6600 4850
@@
 F 0 "J1" H 2200 4850 50  0000 C CNN
 F 1 "Conn_01x05_Female" H 2200 4750 50  0000 C CNN
-F 2 "" H 2300 4400 50  0001 C CNN
+F 2 "kicadlib:SMD_JST_5_PIN_VERT" H 2300 4400 50  0001 C CNN
 F 3 "~" H 2300 4400 50  0001 C CNN
 	1    2300 4400
@@
 Text Label 2500 4200 0    50   ~ 0
 vdd
-Text Label 2500 4300 0    50   ~ 0
+Text Label 2500 4500 0    50   ~ 0
 ~rst
 Text Label 2500 4400 0    50   ~ 0
 swclk
-Text Label 2500 4500 0    50   ~ 0
+Text Label 2500 4300 0    50   ~ 0
 swdio
 $Comp
@@
 swd debug header
 NoConn ~ 5650 3450
-NoConn ~ 5650 3550
 NoConn ~ 5650 3650
 NoConn ~ 5650 3850
@@
 F 0 "R3" V 6493 3750 50  0000 C CNN
 F 1 "R10" V 6584 3750 50  0000 C CNN
-F 2 "" V 6630 3750 50  0001 C CNN
+F 2 "Resistor_SMD:R_0603_1608Metric_Pad1.05x0.95mm_HandSolder" V 6630 3750 50  0001 C CNN
 F 3 "~" H 6700 3750 50  0001 C CNN
 	1    6700 3750
@@
 F 0 "TP1" H 5958 4520 50  0000 L CNN
 F 1 "TestPoint" H 5958 4429 50  0000 L CNN
-F 2 "" H 6100 4400 50  0001 C CNN
+F 2 "kicadlib:TEST_0.100" H 6100 4400 50  0001 C CNN
 F 3 "~" H 6100 4400 50  0001 C CNN
 	1    5900 4400
@@
 F 0 "C1" H 4215 1846 50  0000 L CNN
 F 1 "C" H 4215 1755 50  0000 L CNN
-F 2 "" H 4138 1650 50  0001 C CNN
+F 2 "Capacitor_SMD:C_0603_1608Metric_Pad1.05x0.95mm_HandSolder" H 4138 1650 50  0001 C CNN
 F 3 "~" H 4100 1800 50  0001 C CNN
 	1    4100 1800
@@
 Text Notes 8100 3300 0    50   ~ 0
 rgb led out\nvin nominal 5v\ni/o works with 3.3v
+$Comp
+L Regulator_Linear:MCP1700-3302E_SOT23 U2
+U 1 1 5BA6934A
+P 5400 1550
+F 0 "U2" H 5400 1792 50  0000 C CNN
+F 1 "MCP1700-3302E_SOT23" H 5400 1701 50  0000 C CNN
+F 2 "Package_TO_SOT_SMD:SOT-23" H 5400 1775 50  0001 C CNN
+F 3 "http://ww1.microchip.com/downloads/en/DeviceDoc/20001826C.pdf" H 5400 1550 50  0001 C CNN
+	1    5400 1550
+	1    0    0    -1
+$EndComp
+NoConn ~ 5650 3550
 $EndSCHEMATC
